Commit message: fix(urdf): reorder links/joints, add joint limits & velocities, add middle arm camera mount

File: giava.urdf (robot description, URDF)
Before this commit: robot giava, 29 links, 28 joints
Links:
- added link middlecamera_body, mass 0.04595740741006651; collision mesh filename=interbotix_ws/src/wx250s_7dof_description/meshes/camera_bod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 scale=0.001 0.001 0.001; visual mesh filename=interbotix_ws/src/wx250s_7dof_description/meshes/camera_bod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 scale=0.001 0.001 0.001
- added link middlecamera_cover, mass 0.04595740741006651; collision mesh filename=interbotix_ws/src/wx250s_7dof_description/meshes/camera_cov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 scale=0.001 0.001 0.001; visual mesh filename=interbotix_ws/src/wx250s_7dof_description/meshes/camera_cov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 scale=0.001 0.001 0.001
Joints:
- removed joint middlebase_link_Revolute-3
- added joint middlebase_link: type revolute, parent middlebase_link, child middleshoulder_link, origin xyz=0.0 0.0 0.069 rpy=0.0 -0.0 -1.5707963267948963, axis 0.0 0.0 1.0, limit lower=-3.141582653589793 upper=3.141582653589793 effort=10 velocity=3.141592653589793
- added joint middlecamera_body_fixed: type fixed, parent middlecamera, child middlecamera_body, origin xyz=0.0 0.0 0.0 rpy=0.0 0.0 0.0
- added joint middlecamera_cover_fixed: type fixed, parent middlecamera, child middlecamera_cover, origin xyz=0.0 0.0 0.0 rpy=0.0 0.0 0.0
- joint leftelbow: limit lower=-1.762780 upper=1.605700 -> lower=-1.762780 upper=1.605700 velocity=3.141592653589793
- joint leftforearm_roll: limit lower=-3.141580 upper=3.141580 -> lower=-3.141580 upper=3.141580 velocity=3.141592653589793
- joint leftleft_finger: limit lower=0.000000 upper=0.041000 -> lower=0.000000 upper=0.041000 velocity=3.141592653589793
- joint leftright_finger: limit lower=0.000000 upper=0.041000 -> lower=0.000000 upper=0.041000 velocity=3.141592653589793
- joint leftshoulder: limit lower=-1.850050 upper=1.256640 -> lower=-1.850050 upper=1.256640 velocity=3.141592653589793
- joint leftwaist: limit lower=-3.141580 upper=3.141580 -> lower=-3.141580 upper=3.141580 velocity=3.141592653589793
- joint leftwrist_angle: limit lower=-1.867500 upper=2.234020 -> lower=-1.867500 upper=2.234020 velocity=3.141592653589793
- joint leftwrist_rotate: limit lower=-3.141580 upper=3.141580 -> lower=-3.141580 upper=3.141580 velocity=3.141592653589793
- joint middlelower_forearm_link_Revolute-7: limit (none) -> lower=-1.7453292519943295 upper=2.1467549799530254 effort=5 velocity=3.141592653589793; type continuous -> revolute
- joint middlepan_link_Revolute-2: limit (none) -> lower=-3.141592653589793 upper=3.141592653589793 effort=1 velocity=3.141592653589793; type continuous -> revolute
- joint middleshoulder_link_Revolute-4: limit (none) -> lower=-1.8849555921538759 upper=1.9896753472735358 effort=20 velocity=3.141592653589793; type continuous -> revolute
- joint middleupper_arm_link_Revolute-5: limit (none) -> lower=-2.1467549799530254 upper=1.6057029118347832 effort=15 velocity=3.141592653589793; type continuous -> revolute
- joint middleupper_forearm_link_Revolute-6: limit (none) -> lower=-3.141582653589793 upper=3.141582653589793 effort=2 velocity=3.141592653589793; type continuous -> revolute
- joint middlewrist_link_Revolute-1: limit (none) -> lower=-3.141592653589793 upper=3.141592653589793 effort=1 velocity=3.141592653589793; type continuous -> revolute
- joint rightelbow: limit lower=-1.762780 upper=1.605700 -> lower=-1.762780 upper=1.605700 velocity=3.141592653589793
- joint rightforearm_roll: limit lower=-3.141580 upper=3.141580 -> lower=-3.141580 upper=3.141580 velocity=3.141592653589793
- joint rightleft_finger: limit lower=0.000000 upper=0.041000 -> lower=0.000000 upper=0.041000 velocity=3.141592653589793
- joint rightright_finger: limit lower=0.000000 upper=0.041000 -> lower=0.000000 upper=0.041000 velocity=3.141592653589793
- joint rightshoulder: limit lower=-1.850050 upper=1.256640 -> lower=-1.850050 upper=1.256640 velocity=3.141592653589793
- joint rightwaist: limit lower=-3.141580 upper=3.141580 -> lower=-3.141580 upper=3.141580 velocity=3.141592653589793
- joint rightwrist_angle: limit lower=-1.867500 upper=2.234020 -> lower=-1.867500 upper=2.234020 velocity=3.141592653589793
- joint rightwrist_rotate: limit lower=-3.141580 upper=3.141580 -> lower=-3.141580 upper=3.141580 velocity=3.141592653589793

Commit message: corrected left/right mismatch

File: giava.urdf (robot description, URDF)
Before this commit: robot giava, 31 links, 30 joints
Links:
- link leftleft_finger_link: mass 0.086294 -> 0.086293
- link leftright_finger_link: mass 0.086293 -> 0.086294
- link rightleft_finger_link: mass 0.086294 -> 0.086293
- link rightright_finger_link: mass 0.086293 -> 0.086294
Joints:
- removed joint middlelower_forearm_link_Revolute-7
- removed joint middlepan_link_Revolute-2
- removed joint middleshoulder_link_Revolute-4
- removed joint middleupper_arm_link_Revolute-5
- removed joint middleupper_forearm_link_Revolute-6
- removed joint middlewrist_link_Revolute-1
- added joint middlelower_forearm_link: type revolute, parent middlelower_forearm_link, child middlewrist_link, origin xyz=0.0782 0.0 0.019100000000000002 rpy=1.5707963267949763 -0.0 1.5707963267948966, axis 2.8698592549372254e-42 -1.0 7.97360475549766e-14, limit lower=-1.7453292519943295 upper=2.1467549799530254 effort=5 velocity=3.141592653589793
- added joint middlepan_link: type revolute, parent middlepan_link, child middlecamera, origin xyz=0.04125 0.03725000000000001 1.1379786002407855e-17 rpy=-1.5707963267948963 2.5199808612277694e-29 -1.4272358353620772e-42, axis 0.0 -6.162975822039155e-33 1.0, limit lower=-3.141592653589793 upper=3.141592653589793 effort=1 velocity=3.141592653589793
- added joint middleshoulder_link: type revolute, parent middleshoulder_link, child middleupper_arm_link, origin xyz=0.0 0.013999999999999999 0.04125 rpy=-0.0 -1.5707963267948966 0, axis 0.0 -1.0 0.0, limit lower=-1.8849555921538759 upper=1.9896753472735358 effort=20 velocity=3.141592653589793
- added joint middleupper_arm_link: type revolute, parent middleupper_arm_link, child middleupper_forearm_link, origin xyz=0.25 0.0 -0.05 rpy=2.1791458186645653e-52 -1.4349296274686127e-42 2.8698592549372254e-42, axis -2.8698592549372254e-42 -1.0 -2.1791458186645675e-52, limit lower=-2.1467549799530254 upper=1.6057029118347832 effort=15 velocity=3.141592653589793
- added joint middleupper_forearm_link: type revolute, parent middleupper_forearm_link, child middlelower_forearm_link, origin xyz=0.0 -0.013499999999999998 -0.1718 rpy=1.5707963267948966 1.5707963267948966 0, axis 1.0 -1.4349296274686127e-42 2.1791458186645653e-52, limit lower=-3.141582653589793 upper=3.141582653589793 effort=2 velocity=3.141592653589793
- added joint middlewrist_link: type revolute, parent middlewrist_link, child middlepan_link, origin xyz=-1.7053025658242404e-15 -0.01899999999999482 0.06500000000000149 rpy=-1.570796326794897 -1.5707963267948128 0, axis 1.0 -1.4349446804892014e-42 1.6339707364920764e-13, limit lower=-3.141592653589793 upper=3.141592653589793 effort=1 velocity=3.141592653589793
- joint base_leftbase_link_fixed: origin xyz=-0.469000 -0.019000 0.020000 rpy=0.000000 0.000000 0.000000 -> xyz=0.469000 -0.019000 0.020000 rpy=0.000000 0.000000 3.141593
- joint base_rightbase_link_fixed: origin xyz=0.469000 -0.019000 0.020000 rpy=0.000000 0.000000 3.141593 -> xyz=-0.469000 -0.019000 0.020000 rpy=0.000000 0.000000 0.000000
- joint leftleft_finger: origin xyz=0.019100 -0.014164 0.021173 rpy=-1.570796 0.000000 1.570796 -> xyz=-0.019100 -0.014164 0.021173 rpy=1.570796 0.000000 1.570796
- joint leftright_finger: origin xyz=-0.019100 -0.014164 0.021173 rpy=1.570796 0.000000 1.570796 -> xyz=0.019100 -0.014164 0.021173 rpy=-1.570796 0.000000 1.570796
- joint rightleft_finger: origin xyz=0.019100 -0.014164 0.021173 rpy=-1.570796 0.000000 1.570796 -> xyz=-0.019100 -0.014164 0.021173 rpy=1.570796 0.000000 1.570796
- joint rightright_finger: origin xyz=-0.019100 -0.014164 0.021173 rpy=1.570796 0.000000 1.570796 -> xyz=0.019100 -0.014164 0.021173 rpy=-1.570796 0.000000 1.570796
