Commit message: Pushing code with modular setup to enable left, right, and bimanual data collection, replay, and move

File: giava.urdf (robot description, URDF)
Before this commit: robot giava, 31 links, 30 joints
Joints:
- removed joint middlebase_link
- removed joint middlelower_forearm_link
- removed joint middlepan_link
- removed joint middleshoulder_link
- removed joint middleupper_arm_link
- removed joint middleupper_forearm_link
- removed joint middlewrist_link
- added joint middlebase: type revolute, parent middlebase_link, child middleshoulder_link, origin xyz=0.0 0.0 0.069 rpy=0.0 -0.0 -1.5707963267948963, axis 0.0 0.0 1.0, limit lower=-3.141582653589793 upper=3.141582653589793 effort=10 velocity=3.141592653589793
- added joint middlelower_forearm: type revolute, parent middlelower_forearm_link, child middlewrist_link, origin xyz=0.0782 0.0 0.019100000000000002 rpy=1.5707963267949763 -0.0 1.5707963267948966, axis 2.8698592549372254e-42 -1.0 7.97360475549766e-14, limit lower=-1.7453292519943295 upper=2.1467549799530254 effort=5 velocity=3.141592653589793
- added joint middlepan: type revolute, parent middlepan_link, child middlecamera, origin xyz=0.04125 0.03725000000000001 1.1379786002407855e-17 rpy=-1.5707963267948963 2.5199808612277694e-29 -1.4272358353620772e-42, axis 0.0 -6.162975822039155e-33 1.0, limit lower=-3.141592653589793 upper=3.141592653589793 effort=1 velocity=3.141592653589793
- added joint middleshoulder: type revolute, parent middleshoulder_link, child middleupper_arm_link, origin xyz=0.0 0.013999999999999999 0.04125 rpy=-0.0 -1.5707963267948966 0, axis 0.0 -1.0 0.0, limit lower=-1.8849555921538759 upper=1.9896753472735358 effort=20 velocity=3.141592653589793
- added joint middleupper_arm: type revolute, parent middleupper_arm_link, child middleupper_forearm_link, origin xyz=0.25 0.0 -0.05 rpy=2.1791458186645653e-52 -1.4349296274686127e-42 2.8698592549372254e-42, axis -2.8698592549372254e-42 -1.0 -2.1791458186645675e-52, limit lower=-2.1467549799530254 upper=1.6057029118347832 effort=15 velocity=3.141592653589793
- added joint middleupper_forearm: type revolute, parent middleupper_forearm_link, child middlelower_forearm_link, origin xyz=0.0 -0.013499999999999998 -0.1718 rpy=1.5707963267948966 1.5707963267948966 0, axis 1.0 -1.4349296274686127e-42 2.1791458186645653e-52, limit lower=-3.141582653589793 upper=3.141582653589793 effort=2 velocity=3.141592653589793
- added joint middlewrist: type revolute, parent middlewrist_link, child middlepan_link, origin xyz=-1.7053025658242404e-15 -0.01899999999999482 0.06500000000000149 rpy=-1.570796326794897 -1.5707963267948128 0, axis 1.0 -1.4349446804892014e-42 1.6339707364920764e-13, limit lower=-3.141592653589793 upper=3.141592653589793 effort=1 velocity=3.141592653589793

File: interbotix_ws/src/wx250s_7dof_description/urdf/wx250s_7dof.urdf (robot description, URDF)
Before this commit: robot wx250s, 7 links, 6 joints
Links:
- added link wx250s/camera_yaw_link, mass 0.03; collision mesh filename=package://wx250s_7dof_description/meshes/wx250s_7dof_camera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 scale=0.001 0.001 0.001; visual mesh filename=package://wx250s_7dof_description/meshes/wx250s_7dof_camera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 scale=0.001 0.001 0.001
Joints:
- added joint camera_yaw: type revolute, parent wx250s/camera_roll_link, child wx250s/camera_yaw_link, origin xyz=0 0 0 rpy=0 0 0, axis 0 0 1, limit lower=-3.141592653589793 upper=3.141592653589793 effort=1 velocity=3.141592653589793

Commit message: Latest commit (IK)

File: giava.urdf (robot description, URDF)
Before this commit: robot giava, 31 links, 30 joints
Links:
- link middlecamera_body: geometry collision mesh filename=interbotix_ws/src/wx250s_7dof_description/urdf/meshes/camer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 scale=0.001 0.001 0.001; visual mesh filename=interbotix_ws/src/wx250s_7dof_description/urdf/meshes/camer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 scale=0.001 0.001 0.001
- link middlecamera_cover: geometry collision mesh filename=interbotix_ws/src/wx250s_7dof_description/urdf/meshes/camer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 scale=0.001 0.001 0.001; visual mesh filename=interbotix_ws/src/wx250s_7dof_description/urdf/meshes/camer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 scale=0.001 0.001 0.001

File: interbotix_ws/src/wx250s_7dof_description/urdf/wx250s_7dof.urdf (robot description, URDF)
Before this commit: robot wx250s, 8 links, 7 joints
Links:
- removed link wx250s/base_link
- removed link wx250s/camera_roll_link
- removed link wx250s/camera_yaw_link
- removed link wx250s/lower_forearm_link
- removed link wx250s/shoulder_link
- removed link wx250s/upper_arm_link
- removed link wx250s/upper_forearm_link
- removed link wx250s/wrist_link
- added link 430---Wrist-v3, mass 0.03273465768623896; collision mesh filename=meshes/430---Wrist-v3.stl scale=0.001 0.001 0.001; visual mesh filename=meshes/430---Wrist-v3.stl scale=0.001 0.001 0.001
- added link 430-Base-v3, mass 0.5387615553440656; collision mesh filename=meshes/430-Base-v3.stl scale=0.001 0.001 0.001; visual mesh filename=meshes/430-Base-v3.stl scale=0.001 0.001 0.001
- added link 430-Dual-Shoulder-v2, mass 0.06870346818902391; collision mesh filename=meshes/430-Dual-Shoulder-v2.stl scale=0.001 0.001 0.001; visual mesh filename=meshes/430-Dual-Shoulder-v2.stl scale=0.001 0.001 0.001
- added link SIMPLIFIED---WXA-250-6DOF-Lower-Forearm-v4, mass 0.06645495133905654; collision mesh filename=meshes/SIMPLIFIED---WXA-250-6DOF-Lower-Forearm-v4.stl scale=0.001 0.001 0.001; visual mesh filename=meshes/SIMPLIFIED---WXA-250-6DOF-Lower-Forearm-v4.stl scale=0.001 0.001 0.001
- added link SIMPLIFIED---WXA-250-6DOF-Upper-Forearm-v3, mass 0.05883498167352428; collision mesh filename=meshes/SIMPLIFIED---WXA-250-6DOF-Upper-Forearm-v3.stl scale=0.001 0.001 0.001; visual mesh filename=meshes/SIMPLIFIED---WXA-250-6DOF-Upper-Forearm-v3.stl scale=0.001 0.001 0.001
- added link UA---6---WX-250-v2, mass 0.14814385180189243; collision mesh filename=meshes/UA---6---WX-250-v2.stl scale=0.001 0.001 0.001; visual mesh filename=meshes/UA---6---WX-250-v2.stl scale=0.001 0.001 0.001
- added link gripper_motor, mass 0.03546994534296931; collision mesh filename=meshes/gripper_motor.stl scale=0.001 0.001 0.001; visual mesh filename=meshes/gripper_motor.stl scale=0.001 0.001 0.001
- added link middlecamera, mass 0.06867323298593662; collision mesh filename=meshes/middlecamera.stl scale=0.001 0.001 0.001; visual mesh filename=meshes/middlecamera.stl scale=0.001 0.001 0.001
Joints:
- joint camera_roll: axis 1 0 0 -> 1.0 1.5407439555097887e-33 -1.513396580661073e-36; child wx250s/camera_roll_link -> gripper_motor; limit lower=-3.141592653589793 upper=3.141592653589793 effort=1 velocity=3.141592653589793 -> lower=-2.78 upper=2.99 effort=1 velocity=3.141592653589793; origin xyz=0.065 0 0 rpy=0 0 0 -> xyz=-1.7053025658242404e-15 0.01899999999999482 -0.06500000000000149 rpy=1.5707963267948966 1.5707963267948128 0; parent wx250s/wrist_link -> 430---Wrist-v3
- joint camera_yaw: axis 0 0 1 -> -6.162975822039155e-33 -2.465190328815662e-32 0.9999999999999999; child wx250s/camera_yaw_link -> middlecamera; limit lower=-3.141592653589793 upper=3.141592653589793 effort=1 velocity=3.141592653589793 -> lower=-3.10 upper=3.07 effort=1 velocity=3.141592653589793; origin xyz=0 0 0 rpy=0 0 0 -> xyz=0.04125 0.03725000000000001 0.0 rpy=-1.5707963267948966 9.860300543221678e-33 -4.622231866529366e-33; parent wx250s/camera_roll_link -> gripper_motor
- joint elbow: axis 0 1 0 -> -7.703719777548943e-34 -1.0 -4.898963095872863e-35; child wx250s/upper_forearm_link -> SIMPLIFIED---WXA-250-6DOF-Upper-Forearm-v3; limit lower=-2.1467549799530254 upper=1.6057029118347832 effort=15 velocity=3.141592653589793 -> lower=-2.13 upper=1.60 effort=15 velocity=3.141592653589793; origin xyz=0.04975 0 0.25 rpy=0 0 0 -> xyz=0.25 -0.027999999999999997 -0.05 rpy=3.141592653589793 -0.0 0.0; parent wx250s/upper_arm_link -> UA---6---WX-250-v2
- joint forearm_roll: axis 1 0 0 -> 1.0 1.5407439555097887e-33 -1.513396580661073e-36; child wx250s/lower_forearm_link -> SIMPLIFIED---WXA-250-6DOF-Lower-Forearm-v4; limit lower=-3.141582653589793 upper=3.141582653589793 effort=2 velocity=3.141592653589793 -> lower=-1.58 upper=1.51 effort=2 velocity=3.141592653589793; origin xyz=0.175 0 0 rpy=0 0 0 -> xyz=0.0 -0.014499999999999999 0.1718 rpy=-1.5707963267948966 -1.5707963267948966 0; parent wx250s/upper_forearm_link -> SIMPLIFIED---WXA-250-6DOF-Upper-Forearm-v3
- joint shoulder: axis 0 1 0 -> 7.703719777548943e-34 -1.0 -4.898963060357343e-35; child wx250s/upper_arm_link -> UA---6---WX-250-v2; limit lower=-1.8849555921538759 upper=1.9896753472735358 effort=20 velocity=3.141592653589793 -> lower=-1.92 upper=1.70 effort=20 velocity=3.141592653589793; origin xyz=0 0 0.03865 rpy=0 0 0 -> xyz=-6.357687571391029e-35 0.013999999999999999 0.04125 rpy=-1.1869459682199748e-66 -1.5707963267948966 0; parent wx250s/shoulder_link -> 430-Dual-Shoulder-v2
- joint waist: axis 0 0 1 -> -1.5407439555097887e-33 0.0 1.0; child wx250s/shoulder_link -> 430-Dual-Shoulder-v2; limit lower=-3.141582653589793 upper=3.141582653589793 effort=10 velocity=3.141592653589793 -> lower=-6.35 upper=0.00 effort=10 velocity=3.141592653589793; origin xyz=0 0 0.072 rpy=0 0 0 -> xyz=9.457430695284461e-18 -2.637399261832539e-17 0.06899999988078945 rpy=1.24568280002494e-17 -1.8140360346504614e-19 -1.5707963267948963; parent wx250s/base_link -> 430-Base-v3
- joint wrist_angle: axis 0 1 0 -> 7.703719777548943e-34 -1.0 7.97360475549766e-14; child wx250s/wrist_link -> 430---Wrist-v3; limit lower=-1.7453292519943295 upper=2.1467549799530254 effort=5 velocity=3.141592653589793 -> lower=-1.54 upper=2.12 effort=5 velocity=3.141592653589793; origin xyz=0.075 0 0 rpy=0 0 0 -> xyz=0.0782 0.0 0.019100000000000002 rpy=-1.5707963267948168 -0.0 1.5707963267948966; parent wx250s/lower_forearm_link -> SIMPLIFIED---WXA-250-6DOF-Lower-Forearm-v4

File: interbotix_ws/src/wx250s_7dof_description/urdf/wx250s_7dof.urdf.xacro (robot description, xacro)
@@ -1,5 +1,5 @@
 <?xml version="1.0"?>
 <robot name="wx250s" xmlns:xacro="http://ros.org/wiki/xacro">
-  <xacro:arg name="robot_name" default = "wx250s"/>
+  <xacro:arg name="robot_name" default="wx250s"/>
   <xacro:arg name="base_link_frame" default="base_link"/>
   <xacro:arg name="show_ar_tag" default="false"/>
@@ -28,12 +28,12 @@
       <origin rpy="0 0 ${pi/2}" xyz="0 0 0"/>
       <geometry>
-        <mesh filename="package://interbotix_xsarm_descriptions/meshes/wx250s_meshes/wx250s_1_base.stl" scale="0.001 0.001 0.001"/>
-      </geometry>
-      <material name="interbotix_black"/>
-    </visual>
-    <collision>
-      <origin rpy="0 0 ${pi/2}" xyz="0 0 0"/>
-      <geometry>
-        <mesh filename="package://interbotix_xsarm_descriptions/meshes/wx250s_meshes/wx250s_1_base.stl" scale="0.001 0.001 0.001"/>
+        <mesh filename="package://wx250s_7dof_description/meshes/430-Base-v3.stl" scale="0.001 0.001 0.001"/>
+      </geometry>
+      <material name="interbotix_black"/>
+    </visual>
+    <collision>
+      <origin rpy="0 0 ${pi/2}" xyz="0 0 0"/>
+      <geometry>
+        <mesh filename="package://wx250s_7dof_description/meshes/430-Base-v3.stl" scale="0.001 0.001 0.001"/>
       </geometry>
     </collision>
@@ -46,5 +46,5 @@
   <joint name="waist" type="revolute">
     <axis xyz="0 0 1"/>
-    <limit effort="10" lower="${-pi + pi_offset}" upper="${pi - pi_offset}" velocity="${pi}"/>
+    <limit effort="10" lower="-6.35" upper="0.00" velocity="${pi}"/>
     <origin rpy="0 0 0" xyz="0 0 0.072"/>
     <parent link="$(arg robot_name)/$(arg base_link_frame)"/>
@@ -65,5 +65,5 @@
       <origin rpy="0 0 ${pi/2}" xyz="0 0 -0.003"/>
       <geometry>
-        <mesh filename="package://interbotix_xsarm_descriptions/meshes/wx250s_meshes/wx250s_2_shoulder.stl" scale="0.001 0.001 0.001"/>
+        <mesh filename="package://wx250s_7dof_description/meshes/430-Dual-Shoulder-v2.stl" scale="0.001 0.001 0.001"/>
       </geometry>
       <material name="interbotix_black"/>
@@ -72,5 +72,5 @@
       <origin rpy="0 0 ${pi/2}" xyz="0 0 -0.003"/>
       <geometry>
-        <mesh filename="package://interbotix_xsarm_descriptions/meshes/wx250s_meshes/wx250s_2_shoulder.stl" scale="0.001 0.001 0.001"/>
+        <mesh filename="package://wx250s_7dof_description/meshes/430-Dual-Shoulder-v2.stl" scale="0.001 0.001 0.001"/>
       </geometry>
     </collision>
@@ -83,5 +83,5 @@
   <joint name="shoulder" type="revolute">
     <axis xyz="0 1 0"/>
-    <limit effort="20" lower="${radians(-108)}" upper="${radians(114)}" velocity="${pi}"/>
+    <limit effort="20" lower="-1.92" upper="1.70" velocity="${pi}"/>
     <origin rpy="0 0 0" xyz="0 0 0.03865"/>
     <parent link="$(arg robot_name)/shoulder_link"/>
@@ -102,12 +102,12 @@
       <origin rpy="0 0 ${pi/2}" xyz="0 0 0"/>
       <geometry>
-        <mesh filename="package://interbotix_xsarm_descriptions/meshes/wx250s_meshes/wx250s_3_upper_arm.stl" scale="0.001 0.001 0.001"/>
-      </geometry>
-      <material name="interbotix_black"/>
-    </visual>
-    <collision>
-      <origin rpy="0 0 ${pi/2}" xyz="0 0 0"/>
-      <geometry>
-        <mesh filename="package://interbotix_xsarm_descriptions/meshes/wx250s_meshes/wx250s_3_upper_arm.stl" scale="0.001 0.001 0.001"/>
+        <mesh filename="package://wx250s_7dof_description/meshes/UA---6---WX-250-v2.stl" scale="0.001 0.001 0.001"/>
+      </geometry>
+      <material name="interbotix_black"/>
+    </visual>
+    <collision>
+      <origin rpy="0 0 ${pi/2}" xyz="0 0 0"/>
+      <geometry>
+        <mesh filename="package://wx250s_7dof_description/meshes/UA---6---WX-250-v2.stl" scale="0.001 0.001 0.001"/>
       </geometry>
     </collision>
@@ -120,5 +120,5 @@
   <joint name="elbow" type="revolute">
     <axis xyz="0 1 0"/>
-    <limit effort="15" lower="${radians(-123)}" upper="${radians(92)}" velocity="${pi}"/>
+    <limit effort="15" lower="-2.13" upper="1.60" velocity="${pi}"/>
     <origin rpy="0 0 0" xyz="0.04975 0 0.25"/>
     <parent link="$(arg robot_name)/upper_arm_link"/>
@@ -139,5 +139,5 @@
       <origin rpy="0 0 0" xyz="0 0 0"/>
       <geometry>
-        <mesh filename="package://interbotix_xsarm_descriptions/meshes/wx250s_meshes/wx250s_4_upper_forearm.stl" scale="0.001 0.001 0.001"/>
+        <mesh filename="package://wx250s_7dof_description/meshes/SIMPLIFIED---WXA-250-6DOF-Upper-Forearm-v3.stl" scale="0.001 0.001 0.001"/>
       </geometry>
       <material name="interbotix_black"/>
@@ -146,5 +146,5 @@
       <origin rpy="0 0 0" xyz="0 0 0"/>
       <geometry>
-        <mesh filename="package://interbotix_xsarm_descriptions/meshes/wx250s_meshes/wx250s_4_upper_forearm.stl" scale="0.001 0.001 0.001"/>
+        <mesh filename="package://wx250s_7dof_description/meshes/SIMPLIFIED---WXA-250-6DOF-Upper-Forearm-v3.stl" scale="0.001 0.001 0.001"/>
       </geometry>
     </collision>
@@ -157,5 +157,5 @@
   <joint name="forearm_roll" type="revolute">
     <axis xyz="1 0 0"/>
-    <limit effort="2" lower="${-pi + pi_offset}" upper="${pi - pi_offset}" velocity="${pi}"/>
+    <limit effort="2" lower="-1.58" upper="1.51" velocity="${pi}"/>
     <origin rpy="0 0 0" xyz="0.175 0 0"/>
     <parent link="$(arg robot_name)/upper_forearm_link"/>
@@ -176,5 +176,5 @@
       <origin rpy="${pi} 0 0" xyz="0 0 0"/>
       <geometry>
-        <mesh filename="package://interbotix_xsarm_descriptions/meshes/wx250s_meshes/wx250s_5_lower_forearm.stl" scale="0.001 0.001 0.001"/>
+        <mesh filename="package://wx250s_7dof_description/meshes/SIMPLIFIED---WXA-250-6DOF-Lower-Forearm-v4.stl" scale="0.001 0.001 0.001"/>
       </geometry>
       <material name="interbotix_black"/>
@@ -183,5 +183,5 @@
       <origin rpy="${pi} 0 0" xyz="0 0 0"/>
       <geometry>
-        <mesh filename="package://interbotix_xsarm_descriptions/meshes/wx250s_meshes/wx250s_5_lower_forearm.stl" scale="0.001 0.001 0.001"/>
+        <mesh filename="package://wx250s_7dof_description/meshes/SIMPLIFIED---WXA-250-6DOF-Lower-Forearm-v4.stl" scale="0.001 0.001 0.001"/>
       </geometry>
     </collision>
@@ -192,7 +192,7 @@
     </inertial>
   </link>
- <joint name="wrist_angle" type="revolute">
+  <joint name="wrist_angle" type="revolute">
     <axis xyz="0 1 0"/>
-    <limit effort="5" lower="${radians(-100)}" upper="${radians(123)}" velocity="${pi}"/>
+    <limit effort="5" lower="-1.54" upper="2.12" velocity="${pi}"/>
     <origin rpy="0 0 0" xyz="0.075 0 0"/>
     <parent link="$(arg robot_name)/lower_forearm_link"/>
@@ -213,12 +213,12 @@
       <origin rpy="0 0 ${pi/2}" xyz="0 0 0"/>
       <geometry>
-        <mesh filename="package://interbotix_xsarm_descriptions/meshes/wx250s_meshes/wx250s_6_wrist.stl" scale="0.001 0.001 0.001"/>
-      </geometry>
-      <material name="interbotix_black"/>
-    </visual>
-    <collision>
-      <origin rpy="0 0 ${pi/2}" xyz="0 0 0"/>
-      <geometry>
-        <mesh filename="package://interbotix_xsarm_descriptions/meshes/wx250s_meshes/wx250s_6_wrist.stl" scale="0.001 0.001 0.001"/>
+        <mesh filename="package://wx250s_7dof_description/meshes/430---Wrist-v3.stl" scale="0.001 0.001 0.001"/>
+      </geometry>
+      <material name="interbotix_black"/>
+    </visual>
+    <collision>
+      <origin rpy="0 0 ${pi/2}" xyz="0 0 0"/>
+      <geometry>
+        <mesh filename="package://wx250s_7dof_description/meshes/430---Wrist-v3.stl" scale="0.001 0.001 0.001"/>
       </geometry>
     </collision>
@@ -230,6 +230,6 @@
   </link>
   <joint name="camera_roll" type="revolute">
-    <axis xyz="1 0 0"/>   <!-- roll -->
-    <limit effort="1" lower="${-pi}" upper="${pi}" velocity="${pi}"/>
+    <axis xyz="1 0 0"/>
+    <limit effort="1" lower="-2.78" upper="2.99" velocity="${pi}"/>
     <origin xyz="0.065 0 0" rpy="0 0 0"/>
     <parent link="$(arg robot_name)/wrist_link"/>
@@ -249,12 +249,10 @@
       <origin xyz="0 0 0" rpy="0 0 0"/>
       <geometry>
-        <mesh filename="package://wx250s_7dof_description/meshes/wx250s_7dof_camera_roll.stl"
-              scale="0.001 0.001 0.001"/>
-      </geometry>
-    </visual>
-    <collision>
-      <geometry>
-        <mesh filename="package://wx250s_7dof_description/meshes/wx250s_7dof_camera_roll.stl"
-              scale="0.001 0.001 0.001"/>
+        <mesh filename="package://wx250s_7dof_description/meshes/430---Wrist-v3.stl" scale="0.001 0.001 0.001"/>
+      </geometry>
+    </visual>
+    <collision>
+      <geometry>
+        <mesh filename="package://wx250s_7dof_description/meshes/430---Wrist-v3.stl" scale="0.001 0.001 0.001"/>
       </geometry>
     </collision>
@@ -265,7 +263,7 @@
     </inertial>
   </link>
-  <!-- <joint name="camera_yaw" type="revolute">
+  <joint name="camera_yaw" type="revolute">
     <axis xyz="0 0 1"/>
-    <limit effort="1" lower="${-pi}" upper="${pi}" velocity="${pi}"/>
+    <limit effort="1" lower="-3.10" upper="3.07" velocity="${pi}"/>
     <origin xyz="0 0 0" rpy="0 0 0"/>
     <parent link="$(arg robot_name)/camera_roll_link"/>
@@ -284,12 +282,10 @@
     <visual>
       <geometry>
-        <mesh filename="package://wx250s_7dof_description/meshes/wx250s_7dof_camera_yaw.stl"
-              scale="0.001 0.001 0.001"/>
-      </geometry>
-    </visual>
-    <collision>
-      <geometry>
-        <mesh filename="package://wx250s_7dof_description/meshes/wx250s_7dof_camera_yaw.stl"
-              scale="0.001 0.001 0.001"/>
+        <mesh filename="package://wx250s_7dof_description/meshes/middlecamera.stl" scale="0.001 0.001 0.001"/>
+      </geometry>
+    </visual>
+    <collision>
+      <geometry>
+        <mesh filename="package://wx250s_7dof_description/meshes/middlecamera.stl" scale="0.001 0.001 0.001"/>
       </geometry>
     </collision>
@@ -299,5 +295,5 @@
       <inertia ixx="3e-5" iyy="3e-5" izz="3e-5" ixy="0" ixz="0" iyz="0"/>
     </inertial>
-  </link> -->
+  </link>
   <xacro:if value="${urdf_loc != ''}">
     <xacro:include filename="${urdf_loc}"/>

Commit message: pyroki ik script

File: giava.urdf (robot description, URDF)
Before this commit: robot giava, 31 links, 30 joints
Links:
- link leftleft_finger_link: mass 0.086293 -> 0.086294
- link leftright_finger_link: mass 0.086294 -> 0.086293
- link rightleft_finger_link: mass 0.086293 -> 0.086294
- link rightright_finger_link: mass 0.086294 -> 0.086293
Joints:
- joint leftleft_finger: limit lower=0.000000 upper=0.041000 velocity=3.141592653589793 -> lower=0.000000 upper=0.041000; origin xyz=-0.019100 -0.014164 0.021173 rpy=1.570796 0.000000 1.570796 -> xyz=0.019100 -0.014164 0.021173 rpy=-1.570796 0.000000 1.570796
- joint leftright_finger: limit lower=0.000000 upper=0.041000 velocity=3.141592653589793 -> lower=0.000000 upper=0.041000; origin xyz=0.019100 -0.014164 0.021173 rpy=-1.570796 0.000000 1.570796 -> xyz=-0.019100 -0.014164 0.021173 rpy=1.570796 0.000000 1.570796
- joint rightleft_finger: limit lower=0.000000 upper=0.041000 velocity=3.141592653589793 -> lower=0.000000 upper=0.041000; origin xyz=-0.019100 -0.014164 0.021173 rpy=1.570796 0.000000 1.570796 -> xyz=0.019100 -0.014164 0.021173 rpy=-1.570796 0.000000 1.570796
- joint rightright_finger: limit lower=0.000000 upper=0.041000 velocity=3.141592653589793 -> lower=0.000000 upper=0.041000; origin xyz=0.019100 -0.014164 0.021173 rpy=-1.570796 0.000000 1.570796 -> xyz=-0.019100 -0.014164 0.021173 rpy=1.570796 0.000000 1.570796

Commit message: Fix URDF finger joints for pyroki + refit collision model
Commit 84d3ad1 dropped the velocity attribute from all four gripper finger
joints; pyroki's URDF parser raises on prismatic joints without velocity
limits, so Robot.from_urdf failed for anyone on this branch. Restore the
original velocity=pi attributes (finger left/right mesh swap kept as-is).

The mesh swap moves the right-finger collision meshes between links, so the
frozen sphere decomposition and pair pruning are regenerated against the new
URDF (180 spheres unchanged in count; kept pairs 5884 -> 5917). Suite hash
verified unchanged: 3815490046334af4.

File: giava.urdf (robot description, URDF)
Before this commit: robot giava, 31 links, 30 joints
Joints:
- joint leftleft_finger: limit lower=0.000000 upper=0.041000 -> lower=0.000000 upper=0.041000 velocity=3.141592653589793
- joint leftright_finger: limit lower=0.000000 upper=0.041000 -> lower=0.000000 upper=0.041000 velocity=3.141592653589793
- joint rightleft_finger: limit lower=0.000000 upper=0.041000 -> lower=0.000000 upper=0.041000 velocity=3.141592653589793
- joint rightright_finger: limit lower=0.000000 upper=0.041000 -> lower=0.000000 upper=0.041000 velocity=3.141592653589793
