Commit message: Collision gate, GJK, scene-camera calibration; correct base separation
URDF
  Base x-separation corrected 938 -> 1040 mm centre-to-centre (bases
  +/-0.469 -> +/-0.520). Measured with a ruler and corroborated two ways:
  per-arm gripper-to-own-base reach matches FK to +/-15 mm (so the error was
  base placement, not kinematics), and the plate-to-plate gap predicts
  329 mm vs 305 mm measured, against 228 mm at the old value.
  NOTE anything recorded before this used FK at 938 mm -- world-frame
  quantities spanning both arms in older datasets are ~102 mm too narrow.

  Also carries the earlier link/joint rename to <arm>_<part> and measured
  joint-limit corrections.

Hard inter-arm collision gate  (capsule_gate.py)
  The IK solver's collision term is a soft cost, checked before the clamps
  and on an INSCRIBED sphere model -- it cannot prove separation. The gate
  checks the final clamped command against CIRCUMSCRIBED geometry, so a
  pass proves the meshes are apart.

  It scales the step rather than refusing the tick: a swept binary search
  for the largest safe fraction, so the arms slide up to the boundary and
  stop there. 600 ticks driving at a -136 mm collision never breach the
  margin, settle at exactly the margin with 0.000 mm spread, and retreat
  is always available.

  Per-pair margins: 25 mm structural, 8 mm fingertip-to-fingertip. One
  global margin made two-arm handovers impossible.

GJK from first principles  (gjk.py, multi_capsule.py)
  Exact convex distance via support functions on the Minkowski difference,
  terminating on the duality bracket. Verified exact on analytic cases and
  to 5e-8 against a constrained optimiser over 300 random hull pairs.

  Used as the gate's fine tier over an 8-piece VHACD decomposition with a
  per-link leak correction (build refuses any link whose union does not
  contain its mesh). Measured against the capsule model on a real approach:
  stops 27 mm closer in true geometry, and is FASTER (0.43 vs 0.79 ms/tick)
  because the gate only asks "is separation >= margin", which the duality
  bound settles in one or two iterations.

Collision mode switch  (collision_modes.py)
  python data_collection.py [episode] [--collision sphere|capsule|gjk]
                                      [--mode av|bimanual|left|right|middle]
  The three models do not live at the same layer: spheres are inscribed
  (soft cost only), GJK is non-differentiable (gate only), only capsules
  can be both. Each preset configures both layers coherently and the mode
  is stamped on every episode.

Scene-camera calibration and reconstruction
  calibration/scene_extrinsics.py gives top_scene/low_scene their
  T_base_camera in two stages: board-only camera-to-camera first (no robot,
  so its measurements are independent evidence about the robot), then an
  anchor to the robot whose residual IS the FK disagreement.

  reconstruction/ turns pixels into metres -- epipolar curves,
  triangulation, plane and known-size fallbacks, each with error bars.
  33 ground-truth selftests. Distortion direction is handled explicitly:
  the D405 factory coefficients run pixel->ray, opposite to OpenCV's, and
  are never passed to solvePnP/stereoCalibrate.

  world_view.py --measure adds click-to-3D; capsule_gate_view.py shows the
  gate live against the real arms.

calibration/selftest.py 64/64, reconstruction/selftest.py 33/33.

File: giava.urdf (robot description, URDF)
Before this commit: robot giava, 31 links, 30 joints
Links:
- removed link leftbase_link
- removed link leftgripper_base
- removed link leftgripper_link
- removed link leftleft_finger_link
- removed link leftlower_forearm_link
- removed link leftright_finger_link
- removed link leftshoulder_link
- removed link leftupper_arm_link
- removed link leftupper_forearm_link
- removed link leftwrist_link
- removed link middlebase_link
- removed link middlecamera
- removed link middlecamera_body
- removed link middlecamera_cover
- removed link middlelower_forearm_link
- removed link middlepan_link
- removed link middleshoulder_link
- removed link middleupper_arm_link
- removed link middleupper_forearm_link
- removed link middlewrist_link
- removed link rightbase_link
- removed link rightgripper_base
- removed link rightgripper_link
- removed link rightleft_finger_link
- removed link rightlower_forearm_link
- removed link rightright_finger_link
- removed link rightshoulder_link
- removed link rightupper_arm_link
- removed link rightupper_forearm_link
- removed link rightwrist_link
- added link left_base_link, mass 0.969034; collision mesh filename=aloha_assets/vx300s_1_base.stl scale=0.001 0.001 0.001; visual mesh filename=aloha_assets/vx300s_1_base.stl scale=0.001 0.001 0.001
- added link left_gripper_base, mass 0.421580; collision mesh filename=aloha_assets/d405_solid.stl; collision mesh filename=aloha_assets/vx300s_7_gripper_bar.stl
- added link left_gripper_link, mass 0.251652
- added link left_left_finger_link, mass 0.086294; collision mesh filename=aloha_assets/vx300s_8_custom_finger_left.stl; visual mesh filename=aloha_assets/vx300s_8_custom_finger_left.stl
- added link left_lower_forearm_link, mass 0.414823; collision mesh filename=aloha_assets/vx300s_5_lower_forearm.stl scale=0.001 0.001 0.001; visual mesh filename=aloha_assets/vx300s_5_lower_forearm.stl scale=0.001 0.001 0.001
- added link left_right_finger_link, mass 0.086293; collision mesh filename=aloha_assets/vx300s_8_custom_finger_right.stl; visual mesh filename=aloha_assets/vx300s_8_custom_finger_right.stl
- added link left_shoulder_link, mass 0.798614; collision mesh filename=aloha_assets/vx300s_2_shoulder.stl scale=0.001 0.001 0.001; visual mesh filename=aloha_assets/vx300s_2_shoulder.stl scale=0.001 0.001 0.001
- added link left_upper_arm_link, mass 0.792592; collision mesh filename=aloha_assets/vx300s_3_upper_arm.stl scale=0.001 0.001 0.001; visual mesh filename=aloha_assets/vx300s_3_upper_arm.stl scale=0.001 0.001 0.001
- added link left_upper_forearm_link, mass 0.322228; collision mesh filename=aloha_assets/vx300s_4_upper_forearm.stl scale=0.001 0.001 0.001; visual mesh filename=aloha_assets/vx300s_4_upper_forearm.stl scale=0.001 0.001 0.001
- added link left_wrist_link, mass 0.115395; collision mesh filename=aloha_assets/vx300s_6_wrist.stl scale=0.001 0.001 0.001; visual mesh filename=aloha_assets/vx300s_6_wrist.stl scale=0.001 0.001 0.001
- added link middle_base_link, mass 7.661178396474684; collision mesh filename=wx250s_7dof_assets/middlebase_link.stl scale=0.001 0.001 0.001; visual mesh filename=wx250s_7dof_assets/middlebase_link.stl scale=0.001 0.001 0.001
- added link middle_camera, mass 0.04595740741006651; collision mesh filename=wx250s_7dof_assets/middlecamera.stl scale=0.001 0.001 0.001; visual mesh filename=wx250s_7dof_assets/middlecamera.stl scale=0.001 0.001 0.001
- added link middle_camera_body, mass 0.04595740741006651; collision mesh filename=interbotix_ws/src/wx250s_7dof_description/urdf/meshes/camer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 scale=0.001 0.001 0.001; visual mesh filename=interbotix_ws/src/wx250s_7dof_description/urdf/meshes/camer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 scale=0.001 0.001 0.001
- added link middle_camera_cover, mass 0.04595740741006651; collision mesh filename=interbotix_ws/src/wx250s_7dof_description/urdf/meshes/camer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 scale=0.001 0.001 0.001; visual mesh filename=interbotix_ws/src/wx250s_7dof_description/urdf/meshes/camer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 scale=0.001 0.001 0.001
- added link middle_lower_forearm_link, mass 0.944988061021575; collision mesh filename=wx250s_7dof_assets/middlelower_forearm_link.stl scale=0.001 0.001 0.001; visual mesh filename=wx250s_7dof_assets/middlelower_forearm_link.stl scale=0.001 0.001 0.001
- added link middle_pan_link, mass 0.46675471997634344; collision mesh filename=wx250s_7dof_assets/middlepan_link.stl scale=0.001 0.001 0.001; visual mesh filename=wx250s_7dof_assets/middlepan_link.stl scale=0.001 0.001 0.001
- added link middle_shoulder_link, mass 0.9769619250514205; collision mesh filename=wx250s_7dof_assets/middleshoulder_link.stl scale=0.001 0.001 0.001; visual mesh filename=wx250s_7dof_assets/middleshoulder_link.stl scale=0.001 0.001 0.001
- added link middle_upper_arm_link, mass 2.1066025697961988; collision mesh filename=wx250s_7dof_assets/middleupper_arm_link.stl scale=0.001 0.001 0.001; visual mesh filename=wx250s_7dof_assets/middleupper_arm_link.stl scale=0.001 0.001 0.001
- added link middle_upper_forearm_link, mass 0.8366322468319658; collision mesh filename=wx250s_7dof_assets/middleupper_forearm_link.stl scale=0.001 0.001 0.001; visual mesh filename=wx250s_7dof_assets/middleupper_forearm_link.stl scale=0.001 0.001 0.001
- added link middle_wrist_link, mass 0.469701678611065; collision mesh filename=wx250s_7dof_assets/middlewrist_link.stl scale=0.001 0.001 0.001; visual mesh filename=wx250s_7dof_assets/middlewrist_link.stl scale=0.001 0.001 0.001
- added link right_base_link, mass 0.969034; collision mesh filename=aloha_assets/vx300s_1_base.stl scale=0.001 0.001 0.001; visual mesh filename=aloha_assets/vx300s_1_base.stl scale=0.001 0.001 0.001
- added link right_gripper_base, mass 0.421580; collision mesh filename=aloha_assets/d405_solid.stl; collision mesh filename=aloha_assets/vx300s_7_gripper_bar.stl
- added link right_gripper_link, mass 0.251652
- added link right_left_finger_link, mass 0.086294; collision mesh filename=aloha_assets/vx300s_8_custom_finger_left.stl; visual mesh filename=aloha_assets/vx300s_8_custom_finger_left.stl
- added link right_lower_forearm_link, mass 0.414823; collision mesh filename=aloha_assets/vx300s_5_lower_forearm.stl scale=0.001 0.001 0.001; visual mesh filename=aloha_assets/vx300s_5_lower_forearm.stl scale=0.001 0.001 0.001
- added link right_right_finger_link, mass 0.086293; collision mesh filename=aloha_assets/vx300s_8_custom_finger_right.stl; visual mesh filename=aloha_assets/vx300s_8_custom_finger_right.stl
- added link right_shoulder_link, mass 0.798614; collision mesh filename=aloha_assets/vx300s_2_shoulder.stl scale=0.001 0.001 0.001; visual mesh filename=aloha_assets/vx300s_2_shoulder.stl scale=0.001 0.001 0.001
- added link right_upper_arm_link, mass 0.792592; collision mesh filename=aloha_assets/vx300s_3_upper_arm.stl scale=0.001 0.001 0.001; visual mesh filename=aloha_assets/vx300s_3_upper_arm.stl scale=0.001 0.001 0.001
- added link right_upper_forearm_link, mass 0.322228; collision mesh filename=aloha_assets/vx300s_4_upper_forearm.stl scale=0.001 0.001 0.001; visual mesh filename=aloha_assets/vx300s_4_upper_forearm.stl scale=0.001 0.001 0.001
- added link right_wrist_link, mass 0.115395; collision mesh filename=aloha_assets/vx300s_6_wrist.stl scale=0.001 0.001 0.001; visual mesh filename=aloha_assets/vx300s_6_wrist.stl scale=0.001 0.001 0.001
Joints:
- removed joint base_leftbase_link_fixed
- removed joint base_middlebase_link_fixed
- removed joint base_rightbase_link_fixed
- removed joint leftelbow
- removed joint leftforearm_roll
- removed joint leftgripper_link_leftgripper_base_fixed
- removed joint leftleft_finger
- removed joint leftright_finger
- removed joint leftshoulder
- removed joint leftwaist
- removed joint leftwrist_angle
- removed joint leftwrist_rotate
- removed joint middlebase
- removed joint middlecamera_body_fixed
- removed joint middlecamera_cover_fixed
- removed joint middlelower_forearm
- removed joint middlepan
- removed joint middleshoulder
- removed joint middleupper_arm
- removed joint middleupper_forearm
- removed joint middlewrist
- removed joint rightelbow
- removed joint rightforearm_roll
- removed joint rightgripper_link_rightgripper_base_fixed
- removed joint rightleft_finger
- removed joint rightright_finger
- removed joint rightshoulder
- removed joint rightwaist
- removed joint rightwrist_angle
- removed joint rightwrist_rotate
- added joint base_left_base_link_fixed: type fixed, parent base, child left_base_link, origin xyz=0.520000 -0.019000 0.020000 rpy=0.000000 0.000000 3.141593
- added joint base_middle_base_link_fixed: type fixed, parent base, child middle_base_link, origin xyz=-0.0 0.4 0.020000 rpy=0.000000 0.000000 0.000000
- added joint base_right_base_link_fixed: type fixed, parent base, child right_base_link, origin xyz=-0.520000 -0.019000 0.020000 rpy=0.000000 0.000000 0.000000
- added joint left_elbow: type revolute, parent left_upper_arm_link, child left_upper_forearm_link, origin xyz=0.059550 0.000000 0.300000 rpy=0.000000 0.000000 0.000000, axis 0.000000 1.000000 0.000000, limit lower=-1.762780 upper=1.710420 velocity=3.141592653589793
- added joint left_forearm_roll: type revolute, parent left_upper_forearm_link, child left_lower_forearm_link, origin xyz=0.200000 0.000000 0.000000 rpy=0.000000 0.000000 0.000000, axis 1.000000 0.000000 0.000000, limit lower=-3.141580 upper=3.141580 velocity=3.141592653589793
- added joint left_gripper_link_left_gripper_base_fixed: type fixed, parent left_gripper_link, child left_gripper_base, origin xyz=0.035000 0.000000 0.000000 rpy=-1.570000 0.000796 -1.570796
- added joint left_left_finger: type prismatic, parent left_gripper_base, child left_left_finger_link, origin xyz=0.019100 -0.014164 0.021173 rpy=-1.570796 0.000000 1.570796, axis 0.000000 0.000000 -1.000000, limit lower=0.000000 upper=0.041000 velocity=3.141592653589793
- added joint left_right_finger: type prismatic, parent left_gripper_base, child left_right_finger_link, origin xyz=-0.019100 -0.014164 0.021173 rpy=1.570796 0.000000 1.570796, axis 0.000000 0.000000 -1.000000, limit lower=0.000000 upper=0.041000 velocity=3.141592653589793
- added joint left_shoulder: type revolute, parent left_shoulder_link, child left_upper_arm_link, origin xyz=0.000000 0.000000 0.048050 rpy=0.000000 0.000000 0.000000, axis 0.000000 1.000000 0.000000, limit lower=-1.954770 upper=1.256640 velocity=3.141592653589793
- added joint left_waist: type revolute, parent left_base_link, child left_shoulder_link, origin xyz=0.000000 0.000000 0.079000 rpy=0.000000 0.000000 0.000000, axis 0.000000 0.000000 1.000000, limit lower=-3.141580 upper=3.141580 velocity=3.141592653589793
- added joint left_wrist_angle: type revolute, parent left_lower_forearm_link, child left_wrist_link, origin xyz=0.100000 0.000000 0.000000 rpy=0.000000 0.000000 0.000000, axis 0.000000 1.000000 0.000000, limit lower=-1.867500 upper=2.234020 velocity=3.141592653589793
- added joint left_wrist_rotate: type revolute, parent left_wrist_link, child left_gripper_link, origin xyz=0.069744 0.000000 0.000000 rpy=0.000000 0.000000 0.000000, axis 1.000000 0.000000 0.000000, limit lower=-3.141580 upper=3.141580 velocity=3.141592653589793
- added joint middle_base: type revolute, parent middle_base_link, child middle_shoulder_link, origin xyz=0.0 0.0 0.069 rpy=0.0 -0.0 -1.5707963267948963, axis 0.0 0.0 1.0, limit lower=-3.141582653589793 upper=3.141582653589793 effort=10 velocity=3.141592653589793
- added joint middle_camera_body_fixed: type fixed, parent middle_camera, child middle_camera_body, origin xyz=0.0 0.0 0.0 rpy=0.0 0.0 0.0
- added joint middle_camera_cover_fixed: type fixed, parent middle_camera, child middle_camera_cover, origin xyz=0.0 0.0 0.0 rpy=0.0 0.0 0.0
- added joint middle_lower_forearm: type revolute, parent middle_lower_forearm_link, child middle_wrist_link, origin xyz=0.0782 0.0 0.019100000000000002 rpy=1.5707963267949763 -0.0 1.5707963267948966, axis 2.8698592549372254e-42 -1.0 7.97360475549766e-14, limit lower=-1.7453292519943295 upper=2.1467549799530254 effort=5 velocity=3.141592653589793
- added joint middle_pan: type revolute, parent middle_pan_link, child middle_camera, origin xyz=0.04125 0.03725000000000001 1.1379786002407855e-17 rpy=-1.5707963267948963 2.5199808612277694e-29 -1.4272358353620772e-42, axis 0.0 -6.162975822039155e-33 1.0, limit lower=-3.141592653589793 upper=0.915 effort=1 velocity=3.141592653589793
- added joint middle_shoulder: type revolute, parent middle_shoulder_link, child middle_upper_arm_link, origin xyz=0.0 0.013999999999999999 0.04125 rpy=-0.0 -1.5707963267948966 0, axis 0.0 -1.0 0.0, limit lower=-1.8849555921538759 upper=1.9896753472735358 effort=20 velocity=3.141592653589793
- added joint middle_upper_arm: type revolute, parent middle_upper_arm_link, child middle_upper_forearm_link, origin xyz=0.25 0.0 -0.05 rpy=2.1791458186645653e-52 -1.4349296274686127e-42 2.8698592549372254e-42, axis -2.8698592549372254e-42 -1.0 -2.1791458186645675e-52, limit lower=-2.1467549799530254 upper=1.6057029118347832 effort=15 velocity=3.141592653589793
- added joint middle_upper_forearm: type revolute, parent middle_upper_forearm_link, child middle_lower_forearm_link, origin xyz=0.0 -0.013499999999999998 -0.1718 rpy=1.5707963267948966 1.5707963267948966 0, axis 1.0 -1.4349296274686127e-42 2.1791458186645653e-52, limit lower=-3.141582653589793 upper=3.141582653589793 effort=2 velocity=3.141592653589793
- added joint middle_wrist: type revolute, parent middle_wrist_link, child middle_pan_link, origin xyz=-1.7053025658242404e-15 -0.01899999999999482 0.06500000000000149 rpy=-1.570796326794897 -1.5707963267948128 0, axis 1.0 -1.4349446804892014e-42 1.6339707364920764e-13, limit lower=-3.141592653589793 upper=3.141592653589793 effort=1 velocity=3.141592653589793
- added joint right_elbow: type revolute, parent right_upper_arm_link, child right_upper_forearm_link, origin xyz=0.059550 0.000000 0.300000 rpy=0.000000 0.000000 0.000000, axis 0.000000 1.000000 0.000000, limit lower=-1.762780 upper=1.710420 velocity=3.141592653589793
- added joint right_forearm_roll: type revolute, parent right_upper_forearm_link, child right_lower_forearm_link, origin xyz=0.200000 0.000000 0.000000 rpy=0.000000 0.000000 0.000000, axis 1.000000 0.000000 0.000000, limit lower=-3.141580 upper=3.141580 velocity=3.141592653589793
- added joint right_gripper_link_right_gripper_base_fixed: type fixed, parent right_gripper_link, child right_gripper_base, origin xyz=0.035000 0.000000 0.000000 rpy=-1.570000 0.000796 -1.570796
- added joint right_left_finger: type prismatic, parent right_gripper_base, child right_left_finger_link, origin xyz=0.019100 -0.014164 0.021173 rpy=-1.570796 0.000000 1.570796, axis 0.000000 0.000000 -1.000000, limit lower=0.000000 upper=0.041000 velocity=3.141592653589793
- added joint right_right_finger: type prismatic, parent right_gripper_base, child right_right_finger_link, origin xyz=-0.019100 -0.014164 0.021173 rpy=1.570796 0.000000 1.570796, axis 0.000000 0.000000 -1.000000, limit lower=0.000000 upper=0.041000 velocity=3.141592653589793
- added joint right_shoulder: type revolute, parent right_shoulder_link, child right_upper_arm_link, origin xyz=0.000000 0.000000 0.048050 rpy=0.000000 0.000000 0.000000, axis 0.000000 1.000000 0.000000, limit lower=-1.954770 upper=1.256640 velocity=3.141592653589793
- added joint right_waist: type revolute, parent right_base_link, child right_shoulder_link, origin xyz=0.000000 0.000000 0.079000 rpy=0.000000 0.000000 0.000000, axis 0.000000 0.000000 1.000000, limit lower=-3.141580 upper=3.141580 velocity=3.141592653589793
- added joint right_wrist_angle: type revolute, parent right_lower_forearm_link, child right_wrist_link, origin xyz=0.100000 0.000000 0.000000 rpy=0.000000 0.000000 0.000000, axis 0.000000 1.000000 0.000000, limit lower=-1.867500 upper=2.234020 velocity=3.141592653589793
- added joint right_wrist_rotate: type revolute, parent right_wrist_link, child right_gripper_link, origin xyz=0.069744 0.000000 0.000000 rpy=0.000000 0.000000 0.000000, axis 1.000000 0.000000 0.000000, limit lower=-3.141580 upper=3.141580 velocity=3.141592653589793
